File: CoreDuino.sch (EAGLE design)
At the start: 18 parts, among them U1 ATMEGA328P_TQFP

Commit message: More Changes
More Changes
Parts:
- removed JP1, JP2, JP3, JP4, JP5, JP6, JP7, JP8, JP9: (no value), adafruit:PINHD-1X1CB
- added J1, J10, J11, J12, J13, J14, J15, J17, J18, J19, J2, J20, J21, J22, J23, J24, J25, J3, J4, J5, J6, J8, J9: (no value), SparkFun-Connectors:M01NOSILK-KIT
- added J16: (no value), SparkFun-Connectors:M06NO_SILK_FEMALE_PTH
- added J7: AVR_SPI_PRG_6NS, SparkFun-Connectors:AVR_SPI_PRG_6NS
- added LED1: (no value), adafruit:LEDCHIPLED_0805
- added Y1: 16MHZ, SparkFun-FreqCtrl:RESONATOR16MHZ
Connections:
- net N$2 renamed RESET
- removed net N$4: R2.1, U1.PC4(ADC4/SDA)
- removed net N$5: R3.1, U1.PC5(ADC5/SCL)
- new net A0: J1.1, U1.PC0(ADC0)
- new net A1: J2.1, U1.PC1(ADC1)
- new net A2: J3.1, U1.PC2(ADC2)
- new net A3: J17.1, U1.PC3(ADC3)
- new net A4: J20.1, R2.1, U1.PC4(ADC4/SDA)
- new net A5: J21.1, R3.1, U1.PC5(ADC5/SCL)
- new net A6: J18.1, U1.ADC6
- new net A7: J19.1, U1.ADC7
- new net D10: J6.1, U1.PB2(SS/OC1B)
- new net D2: J11.1, U1.PD2(INT0)
- new net D3: J12.1, U1.PD3(INT1)
- new net D4: J13.1, U1.PD4(XCK/T0)
- new net D5: J14.1, U1.PD5(T1)
- new net D6: J15.1, U1.PD6(AIN0)
- new net D7: J8.1, U1.PD7(AIN1)
- new net D8: J4.1, U1.PB0(ICP)
- new net D9: J5.1, U1.PB1(OC1A)
- new net DTR: C3.2, J16.1
- new net MISO: J7.1, U1.PB4(MISO)
- new net MOSI: J7.4, U1.PB3(MOSI/OC2)
- new net N$2: U1.PB7(XTAL2/TOSC2), Y1.3
- new net RST: J7.5
- new net RXI: J16.3, J9.1, U1.PD0(RXD)
- new net SCK: J7.3, R1.2, U1.PB5(SCK)
- new net TXO: J10.1, J16.2, U1.PD1(TXD)
- net GND: now also J16.5, J16.6, J24.1, J25.1, J7.6, LED1.C, Y1.2
- net N$1: now also LED1.A, R1.1; no longer C3.2
- net N$6: now also U1.PB6(XTAL1/TOSC1), Y1.1; no longer R1.2, U1.PB5(SCK)
- net VCC: now also J16.4, J22.1, J23.1, J7.2
Other:
- note added: "SPI - 6PIN"
